Commit message: completed rough draft of 3D SLIP urdf.

File: mujoco/models/urdf/3D_SLIP.urdf (robot description, URDF)
Before this commit: robot 3D_SLIP, 1 links, 0 joints
Links:
- added link foot, mass 0.1; collision sphere radius=0.025; visual sphere radius=0.025
- added link leg_lower, mass 0.5; visual cylinder length=0.3 radius=0.015
- added link leg_upper, mass 0.5; visual cylinder length=0.3 radius=0.025
- added link x_axis_leg
- added link y_axis_leg
Joints:
- added joint body_to_upper_leg: type fixed, parent y_axis_leg, child leg_upper, origin xyz=0 0 -0.15 rpy=0 0 0, axis 0 1 0
- added joint leg_pitch: type revolute, parent x_axis_leg, child y_axis_leg, origin xyz=0 0 0 rpy=0 0 0, axis 0 1 0, limit lower=-1.5708 upper=1.5708
- added joint leg_prismatic: type prismatic, parent leg_upper, child leg_lower, origin xyz=0 0 -0.15 rpy=0 0 0, axis 0 0 1, limit lower=-0.15 upper=0.15
- added joint leg_roll: type revolute, parent body, child x_axis_leg, origin xyz=0 0 0 rpy=0 0 0, axis 1 0 0, limit lower=-1.5708 upper=1.5708
- added joint leg_to_foot: type fixed, parent leg_lower, child foot, origin xyz=0 0 -0.15 rpy=0 0 0

Commit message: good progress on 3D SLIP xml

File: mujoco/models/urdf/3D_SLIP.urdf (robot description, URDF)
Before this commit: robot 3D_SLIP, 6 links, 5 joints
Links:
- link body: geometry collision sphere radius=0.075; visual mesh filename=../meshes/slip/Body.OBJ

Commit message: goo working XML file

File: mujoco/models/urdf/3D_SLIP.urdf (robot description, URDF)
Before this commit: robot 3D_SLIP, 6 links, 5 joints
Links:
- link leg_lower: mass 0.5 -> 0.1
- link leg_upper: mass 0.5 -> 0.1
- link x_axis_leg: mass None -> 0.001
- link y_axis_leg: mass None -> 0.001
Joints:
- joint body_to_upper_leg: axis 0 1 0 -> (none)
